File: KiCad_files/SignalSniffer/SignalSniffer.kicad_sch (KiCad schematic)
At the start: 27 parts, among them J1 MEM1052-00-283-01-A_REVA, J2 USB4930-00-A, J3 Conn_01x02, U1 ESP32-C6-MINI-1, U2 AP2112K-3.3TRG1, U3 BQ24075QRGTRQ1, U4 TLV9001QDCKRQ1, U5 USBLC6-2SC6

Commit message: changed sd card reader to microsd
Parts:
- added R14, R15, R16: 5.1kR, symbol Device:R
- added R17, R18: 22R, symbol Device:R
- added SW1: SW_Push, symbol Switch:SW_Push
- J1: value MEM1052-00-283-01-A_REVA -> MSD-4-A; footprint MEM1052-00-283-01-A_REVA:GCT_MEM1052-00-283-01-A_REVA -> MSD-4-A
Connections:
- net GND: now also R15.2, R16.2
- net at J2.A5 (CC1): now also R15.1
- net at J2.B5 (CC2): now also R16.1
- net at J1.P1 (CD/DAT3), R10.2: now also U1.26 (IO20)
- net at J1.P2 (CMD), R11.2: no longer U1.16 (IO7)
- net at U5.4 (I/O2): now also R17.1; no longer U1.26 (IO20)
- net at U5.6 (I/O1): now also R18.1; no longer U1.25 (IO19)
- net at J1.P5 (CLK), R12.2: now also U1.27 (IO21); no longer U1.15 (IO6)
- net at J1.P7 (DAT0), R13.2: no longer U1.22 (IO8)
- net at U1.17 (IO12): now also R17.2
- net at U1.18 (IO13): now also R18.2
Other:
- note added: "Number of gpio's and analog inputs to be determined"
- note added: "change connector to MSD-4-A"

Commit message: continued work on esp wiring
Parts:
- removed C3, C5: 10uC, symbol Device:C
- removed C4: 1uC, symbol Device:C
- removed J1: MSD-4-A, MSD-4-A, symbol MEM1052-00-283-01-A:MEM1052-00-283-01-A_REVA
- removed R1: 100kR, symbol Device:R
- removed R14: 5.1kR, symbol Device:R
- removed R2: 15kR, symbol Device:R
- removed R3: 10kR, symbol Device:R
- removed U3: BQ24075QRGTRQ1, RGT16_1P7X1P7_TEX, symbol BQ24075QRGTRQ1:BQ24075QRGTRQ1
- removed U4: TLV9001QDCKRQ1, TLV9001QDCKRQ1:SOT65P210X110-5N, symbol TLV9001QDCKRQ1:TLV9001QDCKRQ1
- added C10, C12, C13, C14, C9: 4.7uC, symbol Device:C
- added C11, C8: 100nC, symbol Device:C
- added C7: 10uC, symbol Device:C
- added D4, D5, D6, D7: LED, symbol Device:LED
- added IC1: BQ24230RGTR, QFN50P300X300X100-17N-D, symbol BQ24230RGTR:BQ24230RGTR
- added IC2, IC3: TSV914AQDRQ1, SOIC127P600X175-14N, symbol TSV914AQDRQ1:TSV914AQDRQ1
- added J4: MSD-4-A, MSD4A, symbol MSD-4-A:MSD-4-A
- added JP2, JP3, JP5, JP6, JP7, JP8: SolderJumper_3_Bridged12, symbol Jumper:SolderJumper_3_Bridged12
- added R19, R20, R21, R25: 10kR, symbol Device:R
- added R22: 3kR, symbol Device:R
- added R26, R27, R36, R37, R39, R41, R42, R44, R45: 100kR, symbol Device:R
- added R28: 0R, symbol Device:R
- added R29, R30, R31, R32: 1kR, symbol Device:R
- added R34: 15kR, symbol Device:R
- added R35, R40, R43: 12kR, symbol Device:R
- added R38: 180kR, symbol Device:R
- added SW2, SW3: SW_SPDT, symbol Switch:SW_SPDT
- added TP1, TP2: TestPoint, symbol Connector:TestPoint
- R10, R13, R5: value 10kR -> 12kR
- R11, R12, R4, R6, R8, R9: value 10kR -> 100kR
- R7: value R -> 12kR
Connections:
- net +3.3V: now also C11.1, C14.1, C7.1, C8.1, IC1.6 (EN1), IC2.4 (V+), IC3.4 (V+), J4.4 (VDD), R19.1, R20.1, R25.1, R29.1, R30.1, R31.1, R32.1; no longer R10.1, R11.1, R12.1, R13.1, R4.1, R5.1, R8.1, R9.1
- net +5V: now also J2.A4 (VBUS), J2.A9 (VBUS), J2.B4 (VBUS), J2.B9 (VBUS), U5.5 (VBUS), C12.1, IC1.13 (IN); no longer U2.1 (VIN)
- net GND: now also J3.2 (Pin_2), R10.2, R12.2, R13.2, R5.2, R9.2, SW1.1, U2.2 (GND), C10.2, C11.2, C12.2, C13.2, C14.2, C7.2, C8.2, C9.2, IC1.15 (TD), IC1.17 (EP), IC1.4 (~{CE}), IC1.5 (EN2), IC1.8 (VSS), IC2.11 (V-), IC3.11 (V-), J4.6 (VSS), J4.G1 (GND_1), J4.G2 (GND_2), J4.G3 (GND_3), J4.G4 (GND_4), R21.2, R22.2, R27.2, R28.1, R34.2, R35.2, R38.2, R39.2, R40.2, R42.2, R43.2, R45.2
- net at J2.SH (SHIELD): now also R28.2
- net at R7.1: now also SW3.3 (C)
- net CS: now reaches U1.26 (IO20)
- net CS: now also J4.2 (CD/DAT3); no longer R10.2
- net at R4.2: now also IC2.3 (+INA), SW2.2 (B)
- net at R11.2: now also IC2.12 (+IND), JP2.2 (C)
- net at R6.1: now also SW2.1 (A)
- net D+: now reaches R18.1, U5.6 (I/O1)
- net at R17.1: now also U1.17 (IO12); no longer U5.4 (I/O2)
- net at J3.1 (Pin_1): now also C9.1, IC1.2 (BAT_1), IC1.3 (BAT_2)
- net D-: now reaches R17.2
- net D-: now also U5.4 (I/O2); no longer U1.17 (IO12)
- net at SW1.2: now also U1.8 (EN), C10.1, R25.2
- net CLK: now reaches U1.27 (IO21)
- net CLK: now also J4.5 (CLK); no longer R12.2
- net at R8.2: now also IC2.5 (+INB), SW3.2 (B)
- net ADC6: now reaches U1.10 (IO5)
- net ADC6: now also IC3.6 (-INB), IC3.7 (OUTB)
- net ADC1: now reaches U1.12 (IO0)
- net ADC1: now also IC2.1 (OUTA), IC2.2 (-INA)
- net ADC2: now reaches U1.13 (IO1)
- net ADC2: now also IC2.6 (-INB), IC2.7 (OUTB)
- net ADC7: now reaches U1.15 (IO6)
- net ADC7: now also IC3.8 (OUTC), IC3.9 (-INC)
- net IO4: now reaches U1.16 (IO7)
- net IO1: now reaches U1.19 (IO14)
- net CardDetect: now reaches U1.20 (IO15)
- net CardDetect: now also J4.CD1
- net LED1: now reaches U1.22 (IO8)
- net LED1: now also D4.1 (K)
- net LED2: now reaches U1.23 (IO9)
- net LED2: now also D5.1 (K)
- net IO2: now reaches U1.24 (IO18)
- net IO3: now reaches U1.25 (IO19)
- net MOSI: now reaches U1.28 (IO22)
- net MOSI: now also J4.3 (CMD)
- net MISO: now reaches U1.29 (IO23)
- net MISO: now also J4.7 (DAT0)
- net at U1.30 (RXD0): now also TP2.1
- net at U1.31 (TXD0): now also TP1.1
- net ADC3: now reaches U1.5 (IO2)
- net ADC3: now also IC2.8 (OUTC), IC2.9 (-INC)
- net ADC4: now reaches U1.6 (IO3)
- net ADC4: now also IC2.13 (-IND), IC2.14 (OUTD)
- net ADC5: now reaches U1.9 (IO4)
- net ADC5: now also IC3.1 (OUTA), IC3.2 (-INA)
- new net: R9.1, SW3.1 (A)
- new net: D7.2 (A), R32.2
- new net: IC1.1 (TS), R21.1
- new net: IC3.3 (+INA), JP8.2 (C), R41.2
- new net: JP8.1 (A), R42.1
- new net: J4.1 (DAT2), R19.2
- new net: JP2.1 (A), R10.1
- new net: R5.1, SW2.3 (C)
- new net: JP5.3 (B), R35.1
- new net: JP3.1 (A), R13.1
- new net: IC2.10 (+INC), JP3.2 (C), R26.2
- new net: JP3.3 (B), R27.1
- new net: D6.2 (A), R31.2
- new net: JP7.3 (B), R43.1
- new net: D5.2 (A), R30.2
- new net: IC1.16 (ISET), R22.1
- new net: JP6.1 (A), R38.1
- new net: IC3.12 (+IND), JP6.2 (C), R36.2
- new net: JP6.3 (B), R34.1
- new net: IC3.10 (+INC), JP5.2 (C), R37.2
- new net: IC3.13 (-IND), IC3.14 (OUTD)
- new net: IC3.5 (+INB), JP7.2 (C), R44.2
- new net: D4.2 (A), R29.2
- new net: JP7.1 (A), R45.1
- new net: JP2.3 (B), R12.1
- new net: JP8.3 (B), R40.1
- new net: JP5.1 (A), R39.1
- new net: J4.8 (DAT1), R20.2
- new net +VDC: C13.1, IC1.10 (OUT_1), IC1.11 (OUT_2), U2.1 (VIN)
- new net AIN1: R4.1
- new net AIN2: R8.1
- new net AIN3: R26.1
- new net AIN4: R11.1
- new net AIN5: R41.1
- new net AIN6: R44.1
- new net AIN7: R37.1
- new net Charging: D7.1 (K), IC1.9 (~{CHG})
- new net PwrGood: D6.1 (K), IC1.7 (~{PGOOD})
- no-connect marks 1 -> 3
Other:
- note added: "+3V3 LDO, check for other LDOs"
- note added: "10k NTC can be used here"
- note added: "Battery Charger And Power-Path Management"
- note added: "Debug & Status LEDs"
- note added: "ESP32-C6"
- note added: "USB-C Receptacle"
- note added: "add connectors"
- note added: "microSD card"
- note added: "undervoltage protection needed"
- note removed: "CS"
- note removed: "Number of gpio's and analog inputs to be determined"
- note removed: "card detect, can be connected to uc"
- note removed: "change connector to MSD-4-A"
- moved on the sheet: J2, R15, R16, R17, R18, SW1, U1, U2, U5

Commit message: added voltage level changers
Parts:
- removed JP2, JP3, JP5, JP6, JP7, JP8: SolderJumper_3_Bridged12, symbol Jumper:SolderJumper_3_Bridged12
- removed R10, R13, R35, R40, R43, R5, R7: 12kR, symbol Device:R
- removed R11, R12, R26, R27, R36, R37, R39, R4, R41, R42, R44, R45, R6, R8, R9: 100kR, symbol Device:R
- removed R34: 15kR, symbol Device:R
- removed R38: 180kR, symbol Device:R
- removed SW2, SW3: SW_SPDT, symbol Switch:SW_SPDT
- added JP10, JP11, JP12, JP4, JP9: SolderJumper_3_Bridged12, symbol Jumper:SolderJumper_3_Bridged12
- added R14, R23, R48, R51, R54, R57, R60: 12kR, symbol Device:R
- added R24, R33, R46, R47, R49, R50, R52, R53, R55, R56, R58, R59, R61, R62: 100kR, symbol Device:R
- added SW4, SW5: SW_SPDT, symbol Switch:SW_SPDT
Connections:
- net AIN1: now also R24.1
- net AIN2: now also R33.1
- net AIN3: now also R52.1
- net AIN4: now also R49.1
- net AIN5: now also R55.1
- net AIN6: now also R58.1
- net AIN7: now also R61.1
- net GND: now also R14.2, R23.2, R46.2, R47.2, R48.2, R50.2, R51.2, R53.2, R54.2, R56.2, R57.2, R59.2, R60.2, R62.2
- net BuffIn2: now reaches IC2.5 (+INB)
- net BuffIn2: now also R33.2, SW5.2 (B)
- net BuffIn5: now reaches IC3.3 (+INA)
- net BuffIn5: now also JP10.2 (C), R55.2
- net BuffIn1: now reaches IC2.3 (+INA)
- net BuffIn1: now also R24.2, SW4.2 (B)
- net BuffIn3: now reaches IC2.10 (+INC)
- net BuffIn3: now also JP9.2 (C), R52.2
- net BuffIn4: now reaches IC2.12 (+IND)
- net BuffIn4: now also JP4.2 (C), R49.2
- net BuffIn7: now reaches IC3.10 (+INC)
- net BuffIn7: now also JP12.2 (C), R61.2
- net BuffIn6: now reaches IC3.5 (+INB)
- net BuffIn6: now also JP11.2 (C), R58.2
- new net: JP10.1 (A), R56.1
- new net: JP10.3 (B), R54.1
- new net: JP9.1 (A), R51.1
- new net: JP9.3 (B), R53.1
- new net: JP12.1 (A), R62.1
- new net: JP12.3 (B), R60.1
- new net: R47.1, SW5.1 (A)
- new net: R23.1, SW5.3 (C)
- new net: JP11.1 (A), R59.1
- new net: R46.1, SW4.1 (A)
- new net: R14.1, SW4.3 (C)
- new net: JP11.3 (B), R57.1
- new net: JP4.1 (A), R48.1
- new net: JP4.3 (B), R50.1
Other:
- note added: "Annotade the schematic!!"
- moved on the sheet: C11, C6, D4, D5, D6, D7, IC2, IC3, R29, R30, R31, R32

Commit message: finished schematic mostly
Parts:
- removed C12, C13, C14, C9: 4.7uC, symbol Device:C
- added C1, C2, C5, C6, C7, C8: 10uC, Capacitor_SMD:C_0402_1005Metric, symbol Device:C
- added J3: 1706013, 1706013:PHOENIX_1706013, symbol Connector:Conn_01x02_Socket
- added J5: 1706013, 1706013:PHOENIX_1706013, symbol Connector:Conn_01x11_Socket
- added JP6, JP7, JP8, JP9: SolderJumper_3_Bridged12, symbol Jumper:SolderJumper_3_Bridged12
- added R25, R26, R27, R28: 100kR, Resistor_SMD:R_0603_1608Metric, symbol Device:R
- added R33, R35, R37, R39: 15kR, Resistor_SMD:R_0603_1608Metric, symbol Device:R
- added R34, R36, R38, R40: 180kR, Resistor_SMD:R_0603_1608Metric, symbol Device:R
- C10: value 4.7uC -> 10uC; footprint (none) -> Capacitor_SMD:C_0402_1005Metric
- C11: footprint (none) -> Capacitor_SMD:C_0805_2012Metric
- C12: renamed from C7; footprint (none) -> Capacitor_SMD:C_0402_1005Metric
- C13: renamed from C8; footprint (none) -> Capacitor_SMD:C_0805_2012Metric
- C3: renamed from C1; footprint (none) -> Capacitor_SMD:C_0402_1005Metric
- C4: renamed from C2; footprint (none) -> Capacitor_SMD:C_0805_2012Metric
- C9: renamed from C6; footprint (none) -> Capacitor_SMD:C_0805_2012Metric
- D1: renamed from D6; footprint (none) -> LED_SMD:LED_0805_2012Metric
- D2: renamed from D7; footprint (none) -> LED_SMD:LED_0805_2012Metric
- D3: renamed from D4; footprint (none) -> LED_SMD:LED_0805_2012Metric
- D4: renamed from D5; footprint (none) -> LED_SMD:LED_0805_2012Metric
- IC1: footprint QFN50P300X300X100-17N-D -> SignalSniffer:QFN50P300X300X100-17N-D
- IC2, IC3: footprint SOIC127P600X175-14N -> SignalSniffer:TSV914AQDRQ1
- J4: footprint MSD4A -> SignalSniffer:MSD4A
- R1: renamed from R15; footprint (none) -> Resistor_SMD:R_0603_1608Metric
- R10: renamed from R14; footprint (none) -> Resistor_SMD:R_0603_1608Metric
- R11: renamed from R46; footprint (none) -> Resistor_SMD:R_0603_1608Metric
- R12: renamed from R23; footprint (none) -> Resistor_SMD:R_0603_1608Metric
- R13: renamed from R47; footprint (none) -> Resistor_SMD:R_0603_1608Metric
- R14: renamed from R51; footprint (none) -> Resistor_SMD:R_0603_1608Metric
- R15: renamed from R53; footprint (none) -> Resistor_SMD:R_0603_1608Metric
- R16: renamed from R48; footprint (none) -> Resistor_SMD:R_0603_1608Metric
- R17: renamed from R50; footprint (none) -> Resistor_SMD:R_0603_1608Metric
- R18: renamed from R54; footprint (none) -> Resistor_SMD:R_0603_1608Metric
- R19: renamed from R56; footprint (none) -> Resistor_SMD:R_0603_1608Metric
- R2: renamed from R24; footprint (none) -> Resistor_SMD:R_0603_1608Metric
- R20: renamed from R57; footprint (none) -> Resistor_SMD:R_0603_1608Metric
- R21: renamed from R59; footprint (none) -> Resistor_SMD:R_0603_1608Metric
- R22: renamed from R60; footprint (none) -> Resistor_SMD:R_0603_1608Metric
- R23: renamed from R62; footprint (none) -> Resistor_SMD:R_0603_1608Metric
- R24: renamed from R28; footprint (none) -> Resistor_SMD:R_0603_1608Metric
- R29: renamed from R22; footprint (none) -> Resistor_SMD:R_0603_1608Metric
- R3: renamed from R33; footprint (none) -> Resistor_SMD:R_0603_1608Metric
- R30: renamed from R25; footprint (none) -> Resistor_SMD:R_0603_1608Metric
- R31: renamed from R17; footprint (none) -> Resistor_SMD:R_0603_1608Metric
- R32: renamed from R18; footprint (none) -> Resistor_SMD:R_0603_1608Metric
- R4: renamed from R52; footprint (none) -> Resistor_SMD:R_0603_1608Metric
- R41: renamed from R21; footprint (none) -> Resistor_SMD:R_0603_1608Metric
- R42: renamed from R19; footprint (none) -> Resistor_SMD:R_0603_1608Metric
- R43: renamed from R20; footprint (none) -> Resistor_SMD:R_0603_1608Metric
- R44: renamed from R31; footprint (none) -> Resistor_SMD:R_0603_1608Metric
- R45: renamed from R32; footprint (none) -> Resistor_SMD:R_0603_1608Metric
- R46: renamed from R29; footprint (none) -> Resistor_SMD:R_0603_1608Metric
- R47: renamed from R30; footprint (none) -> Resistor_SMD:R_0603_1608Metric
- R5: renamed from R49; footprint (none) -> Resistor_SMD:R_0603_1608Metric
- R6: renamed from R55; footprint (none) -> Resistor_SMD:R_0603_1608Metric
- R7: renamed from R58; footprint (none) -> Resistor_SMD:R_0603_1608Metric
- R8: renamed from R61; footprint (none) -> Resistor_SMD:R_0603_1608Metric
- R9: renamed from R16; footprint (none) -> Resistor_SMD:R_0603_1608Metric
- U1: renamed from U2; footprint SOT_RG1_DIO -> SignalSniffer:AP2112K-3.3TRG1
- renumbered J2 to J1, J3 to J2, JP9 to JP1, JP4 to JP2, JP10 to JP3, JP11 to JP4, JP12 to JP5, SW4 to SW1, SW5 to SW2, SW1 to SW3, U5 to U2, U1 to U3
Connections:
- net +3.3V: now also C10.1, C2.1, C8.1
- net +5V: now also J3.1 (Pin_1); no longer IC1.13 (IN)
- net +VDC: now also U1.3 (EN), C1.1
- net AIN1: now also J5.11 (Pin_11)
- net AIN2: now also J5.10 (Pin_10)
- net AIN3: now also J5.9 (Pin_9)
- net AIN4: now also J5.8 (Pin_8)
- net AIN5: now also J5.7 (Pin_7)
- net AIN6: now also J5.6 (Pin_6)
- net AIN7: now also J5.5 (Pin_5)
- net GND: now also C1.2, C2.2, C5.2, C6.2, C7.2, C8.2, J3.2 (Pin_2), R33.2, R34.2, R35.2, R36.2, R37.2, R38.2, R39.2, R40.2
- net IO1: now also JP6.2 (C), R25.2
- net IO2: now also JP7.2 (C), R26.2
- net IO3: now also JP8.2 (C), R27.2
- net IO4: now also IC3.13 (-IND), IC3.14 (OUTD)
- net at IC1.2 (BAT_1), IC1.3 (BAT_2), J2.1 (Pin_1): now also C7.1
- net BuffIn8: now reaches IC3.12 (+IND)
- net BuffIn8: now also JP9.2 (C), R28.2
- net at R30.2, SW3.2, U3.8 (EN): now also C6.1; no longer C10.1
- new net: JP8.1 (A), R38.1
- new net: JP7.1 (A), R36.1
- new net: JP7.3 (B), R35.1
- new net: JP6.1 (A), R34.1
- new net: JP6.3 (B), R33.1
- new net: JP9.3 (B), R39.1
- new net: JP8.3 (B), R37.1
- new net: JP9.1 (A), R40.1
- new net: C5.1, IC1.13 (IN)
- new net DIN1: J5.1 (Pin_1), R25.1
- new net DIN2: J5.2 (Pin_2), R26.1
- new net DIN3: J5.3 (Pin_3), R27.1
- new net DIN4: J5.4 (Pin_4), R28.1
Other:
- note added: "Analog Sense Attenuation"
- note added: "Digital Sense Attenuation"
- note added: "Sense and Power Headers"
- note removed: "Annotade the schematic!!"
- note removed: "add connectors"
- note removed: "undervoltage protection needed"
- moved on the sheet: C11, C12, C13, C3, C4, C9, D1, D2, D3, D4, IC1, IC2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

Commit message: small fixes
Parts:
- added BT1: Battery_Cell, symbol Device:Battery_Cell
Changed lines of the file:
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@@
 	(wire
 		(pts
+			(xy 64.77 161.29) (xy 64.77 163.83)
+		)
+		(stroke
+			(width 0)
+			(type default)
+		)
+	)
+	(wire
+		(pts
 			(xy 115.57 143.51) (xy 129.54 143.51)
 		)
@@
 	(wire
 		(pts
+			(xy 64.77 166.37) (xy 64.77 168.91)
+		)
+		(stroke
+			(width 0)
+			(type default)
+		)
+	)
+	(wire
+		(pts
 			(xy 104.14 68.58) (xy 109.22 68.58)
 		)
@@
 	(wire
 		(pts
+			(xy 64.77 166.37) (xy 68.58 166.37)
+		)
+		(stroke
+			(width 0)
+			(type default)
+		)
+	)
+	(wire
+		(pts
 			(xy 336.55 204.47) (xy 331.47 204.47)
 		)
@@
 	(wire
 		(pts
+			(xy 58.42 168.91) (xy 64.77 168.91)
+		)
+		(stroke
+			(width 0)
+			(type default)
+		)
+	)
+	(wire
+		(pts
 			(xy 162.56 154.94) (xy 168.91 154.94)
 		)
@@
 	(wire
 		(pts
+			(xy 64.77 163.83) (xy 68.58 163.83)
+		)
+		(stroke
+			(width 0)
+			(type default)
+		)
+	)
+	(wire
+		(pts
 			(xy 93.98 71.12) (xy 96.52 71.12)
 		)
@@
 	(wire
 		(pts
+			(xy 58.42 161.29) (xy 64.77 161.29)
+		)
+		(stroke
+			(width 0)
+			(type default)
+		)
+	)
+	(wire
+		(pts
 			(xy 287.02 133.35) (xy 287.02 137.16)
 		)
@@
 					(unit 1)
 				)
+			)
+		)
+	)
+	(symbol
+		(lib_id "Device:Battery_Cell")
+		(at 58.42 166.37 0)
+		(mirror y)
+		(unit 1)
+		(body_style 1)
+		(exclude_from_sim no)
+		(in_bom yes)
+		(on_board no)
+		(in_pos_files yes)
+		(dnp no)
+		(property "Reference" "BT1"
+			(at 52.832 169.164 0)
+			(show_name no)
+			(do_not_autoplace no)
+			(effects
+				(font
+					(size 1.27 1.27)
+				)
+				(justify right)
+			)
+		)
+		(property "Value" "Battery_Cell"
+			(at 52.832 171.704 0)
+			(show_name no)
+			(do_not_autoplace no)
+			(effects
+				(font
+					(size 1.27 1.27)
+				)
+				(justify right)
+			)
+		)
+		(property "Footprint" ""
+			(at 58.42 164.846 90)
+			(hide yes)
+			(show_name no)
+			(do_not_autoplace no)
+			(effects
+				(font
+					(size 1.27 1.27)
+				)
+			)
+		)
+		(property "Datasheet" ""
+			(at 58.42 164.846 90)
+			(hide yes)
+			(show_name no)
+			(do_not_autoplace no)
+			(effects
+				(font
+					(size 1.27 1.27)
+				)
+			)
+		)
+		(property "Description" "Single-cell battery"
+			(at 58.42 166.37 0)
+			(hide yes)
+			(show_name no)
+			(do_not_autoplace no)
+			(effects
+				(font
+					(size 1.27 1.27)
+				)
+			)
+		)
+		(property "Sim.Device" "V"
+			(at 58.42 166.37 0)
+			(hide yes)
+			(show_name no)
+			(do_not_autoplace no)
+			(effects
+				(font
+					(size 1.27 1.27)
+				)
+			)
+		)
+		(property "Sim.Type" "DC"
+			(at 58.42 166.37 0)
+			(hide yes)
+			(show_name no)
+			(do_not_autoplace no)
+			(effects
+				(font
+					(size 1.27 1.27)
+				)
+			)
+		)
+		(property "Sim.Pins" "1=+ 2=-"
+			(at 58.42 166.37 0)
+			(hide yes)
+			(show_name no)
+			(do_not_autoplace no)
+			(effects
+				(font
+					(size 1.27 1.27)
+				)
+			)
+		)
+		(pin "2"
+		)
+		(pin "1"
+		)
+		(instances
+			(project "SignalSniffer"
+				(path "/ce92c05a-4c61-49b6-a2e3-503bb2372f0d"
+					(reference "BT1")
+					(unit 1)
+				)
